File: Ayden/Schematics/PCB/STM.kicad_sch (KiCad schematic)
At the start: 4 parts, among them J1 Screw_Terminal_01x12, U1 NUCLEO-F103RB, U2 NRF24L01_Breakout

Commit message: Update schematic/PCB to include connection for common GND
Parts:
- removed J1: Screw_Terminal_01x12, TerminalBlock_Phoenix:TerminalBlock_Phoenix_PT-1,5-12-3.5-H_1x12_P3.50mm_Horizontal, symbol Connector:Screw_Terminal_01x12
- added J1: Screw_Terminal_01x13, TerminalBlock_Phoenix:TerminalBlock_Phoenix_PT-1,5-13-5.0-H_1x13_P5.00mm_Horizontal, symbol Connector:Screw_Terminal_01x13
Connections:
- net GND: now also J1.13 (Pin_13)
- net at U1.CN7_28 (PA0): now also J1.5 (Pin_5)
- net at U1.CN7_30 (PA1): now also J1.6 (Pin_6)
- net at RN1.4 (R2.2), U1.CN7_35 (PC2): now also J1.2 (Pin_2)
- net at RN1.2 (R1.2), U1.CN7_36 (PC1): now also J1.1 (Pin_1)
- net at RN1.6 (R3.2), U1.CN7_37 (PC3): now also J1.3 (Pin_3)
- net at U1.CN7_38 (PC0): now also J1.7 (Pin_7)
- net at U1.CN10_29 (PB5): now also J1.10 (Pin_10)
- net at U1.CN10_17 (PB6): now also J1.11 (Pin_11)
- net at U1.CN10_21 (PA9): now also J1.12 (Pin_12)
- net at RN1.8 (R4.2), U1.CN10_34 (PC4): now also J1.4 (Pin_4)
- net at U1.CN10_3 (PB8): now also J1.8 (Pin_8)
- net at U1.CN10_27 (PB4): now also J1.9 (Pin_9)
Changed lines of the file:
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@@
+    (stroke (width 0) (type default) (color 0 0 0 0))
+  )
+  (wire (pts (xy 33.02 104.14) (xy 33.02 107.95))
     (stroke (width 0) (type default) (color 0 0 0 0))
   )
@@
   (wire (pts (xy 92.71 49.53) (xy 35.56 49.53))
     (stroke (width 0) (type default) (color 0 0 0 0))
+  )
+  (symbol (lib_id "Connector:Screw_Terminal_01x13") (at 27.94 88.9 0) (mirror y) (unit 1)
+    (in_bom yes) (on_board yes) (fields_autoplaced)
+    (property "Reference" "J1" (id 0) (at 27.94 67.31 0))
+    (property "Value" "Screw_Terminal_01x13" (id 1) (at 27.94 69.85 0))
+    (property "Footprint" "TerminalBlock_Phoenix:TerminalBlock_Phoenix_PT-1,5-13-5.0-H_1x13_P5.00mm_Horizontal" (id 2) (at 27.94 88.9 0)
+      (effects (font (size 1.27 1.27)) hide)
+    )
+    (property "Datasheet" "~" (id 3) (at 27.94 88.9 0)
+      (effects (font (size 1.27 1.27)) hide)
+    )
+    (pin "1")
+    (pin "10")
+    (pin "11")
+    (pin "12")
+    (pin "13")
+    (pin "2")
+    (pin "3")
+    (pin "4")
+    (pin "5")
+    (pin "6")
+    (pin "7")
+    (pin "8")
+    (pin "9")
   )
   (symbol (lib_id "power:+3.3V") (at 266.7 38.1 0) (unit 1)
@@
     (pin "8")
   )
-  (symbol (lib_id "Connector:Screw_Terminal_01x12") (at 27.94 86.36 0) (mirror y) (unit 1)
-    (in_bom yes) (on_board yes) (fields_autoplaced)
-    (property "Reference" "J1" (id 0) (at 27.94 67.31 0))
-    (property "Value" "Screw_Terminal_01x12" (id 1) (at 27.94 69.85 0))
-    (property "Footprint" "TerminalBlock_Phoenix:TerminalBlock_Phoenix_PT-1,5-12-3.5-H_1x12_P3.50mm_Horizontal" (id 2) (at 27.94 86.36 0)
-      (effects (font (size 1.27 1.27)) hide)
-    )
-    (property "Datasheet" "~" (id 3) (at 27.94 86.36 0)
-      (effects (font (size 1.27 1.27)) hide)
-    )
-    (pin "1")
-    (pin "10")
-    (pin "11")
-    (pin "12")
-    (pin "2")
-    (pin "3")
-    (pin "4")
-    (pin "5")
-    (pin "6")
-    (pin "7")
-    (pin "8")
-    (pin "9")
+  (symbol (lib_id "power:GND") (at 33.02 107.95 0) (unit 1)
+    (in_bom yes) (on_board yes) (fields_autoplaced)
+    (property "Reference" "#PWR?" (id 0) (at 33.02 114.3 0)
+      (effects (font (size 1.27 1.27)) hide)
+    )
+    (property "Value" "GND" (id 1) (at 33.02 113.03 0))
+    (property "Footprint" "" (id 2) (at 33.02 107.95 0)
+      (effects (font (size 1.27 1.27)) hide)
+    )
+    (property "Datasheet" "" (id 3) (at 33.02 107.95 0)
+      (effects (font (size 1.27 1.27)) hide)
+    )
+    (pin "1")
   )
   (symbol (lib_id "NUCLEO-F303RE:NUCLEO-F303RE") (at 241.3 36.83 0) (mirror x) (unit 3)
@@
       (reference "#PWR?") (unit 1) (value "+3.3V") (footprint "")
     )
+    (path "/48f6ad6c-0562-4094-aa01-87fd4289ac23"
+      (reference "#PWR?") (unit 1) (value "GND") (footprint "")
+    )
     (path "/8e3c631e-a6bf-431c-83f8-ad67b2db945e"
       (reference "#PWR?") (unit 1) (value "+3.3V") (footprint "")
@@
       (reference "#PWR?") (unit 1) (value "GND") (footprint "")
     )
-    (path "/53648bea-0933-467d-8a5e-b142cc9d5a95"
-      (reference "J1") (unit 1) (value "Screw_Terminal_01x12") (footprint "TerminalBlock_Phoenix:TerminalBlock_Phoenix_PT-1,5-12-3.5-H_1x12_P3.50mm_Horizontal")
+    (path "/0066d758-ac0c-4991-8962-e2aa01cf1795"
+      (reference "J1") (unit 1) (value "Screw_Terminal_01x13") (footprint "TerminalBlock_Phoenix:TerminalBlock_Phoenix_PT-1,5-13-5.0-H_1x13_P5.00mm_Horizontal")
     )
     (path "/89bd5112-d545-404c-9735-0769ab27a22b"
