File: Ayden/Schematics/STM/STM.kicad_sch (KiCad schematic)
At the start: 31 parts, among them U1 STM32F103RBTx, U2 NRF24L01_Breakout

Commit message: Updated schematic for project demo
Parts:
- U1: value STM32F103RBTx -> STM32F103RB
Other:
- note added: "Pressure Mat"
- note added: "To RPi GND"
- note added: "To RPi GPIO1"
Changed lines of the file:
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@@
   (junction (at 31.75 34.29) (diameter 0) (color 0 0 0 0)
   )
+  (junction (at 226.06 102.87) (diameter 0) (color 0 0 0 0)
+  )
   (junction (at 20.32 81.28) (diameter 0) (color 0 0 0 0)
   )
@@
   (junction (at 68.58 60.96) (diameter 0) (color 0 0 0 0)
   )
-  (junction (at 111.76 76.2) (diameter 0) (color 0 0 0 0)
-  )
   (junction (at 20.32 110.49) (diameter 0) (color 0 0 0 0)
   )
@@
   (junction (at 68.58 52.07) (diameter 0) (color 0 0 0 0)
   )
+  (junction (at 104.14 17.78) (diameter 0) (color 0 0 0 0)
+  )
   (junction (at 53.34 104.14) (diameter 0) (color 0 0 0 0)
   )
@@
     (stroke (width 0) (type default) (color 0 0 0 0))
   )
-  (wire (pts (xy 111.76 76.2) (xy 113.03 76.2))
+  (wire (pts (xy 104.14 76.2) (xy 113.03 76.2))
     (stroke (width 0) (type default) (color 0 0 0 0))
   )
@@
     (stroke (width 0) (type default) (color 0 0 0 0))
   )
-  (wire (pts (xy 194.31 72.39) (xy 194.31 46.99))
-    (stroke (width 0) (type default) (color 0 0 0 0))
-  )
   (wire (pts (xy 24.13 118.11) (xy 38.1 118.11))
     (stroke (width 0) (type default) (color 0 0 0 0))
@@
     (stroke (width 0) (type default) (color 0 0 0 0))
   )
+  (wire (pts (xy 226.06 46.99) (xy 110.49 46.99))
+    (stroke (width 0) (type default) (color 0 0 0 0))
+  )
   (wire (pts (xy 34.29 96.52) (xy 34.29 81.28))
     (stroke (width 0) (type default) (color 0 0 0 0))
@@
     (stroke (width 0) (type default) (color 0 0 0 0))
   )
+  (wire (pts (xy 194.31 72.39) (xy 194.31 17.78))
+    (stroke (width 0) (type default) (color 0 0 0 0))
+  )
   (wire (pts (xy 17.78 17.78) (xy 26.67 17.78))
     (stroke (width 0) (type default) (color 0 0 0 0))
@@
     (stroke (width 0) (type default) (color 0 0 0 0))
   )
-  (wire (pts (xy 194.31 46.99) (xy 109.22 46.99))
-    (stroke (width 0) (type default) (color 0 0 0 0))
-  )
   (wire (pts (xy 176.53 118.11) (xy 176.53 160.02))
     (stroke (width 0) (type default) (color 0 0 0 0))
@@
     (stroke (width 0) (type default) (color 0 0 0 0))
   )
-  (wire (pts (xy 106.68 17.78) (xy 106.68 76.2))
+  (wire (pts (xy 226.06 102.87) (xy 226.06 46.99))
+    (stroke (width 0) (type default) (color 0 0 0 0))
+  )
+  (wire (pts (xy 104.14 17.78) (xy 104.14 76.2))
     (stroke (width 0) (type default) (color 0 0 0 0))
   )
@@
     (stroke (width 0) (type default) (color 0 0 0 0))
   )
+  (wire (pts (xy 153.67 87.63) (xy 153.67 107.95))
+    (stroke (width 0) (type default) (color 0 0 0 0))
+  )
+  (wire (pts (xy 148.59 87.63) (xy 153.67 87.63))
+    (stroke (width 0) (type default) (color 0 0 0 0))
+  )
   (wire (pts (xy 39.37 30.48) (xy 39.37 36.83))
     (stroke (width 0) (type default) (color 0 0 0 0))
@@
     (stroke (width 0) (type default) (color 0 0 0 0))
   )
-  (wire (pts (xy 111.76 40.64) (xy 111.76 76.2))
-    (stroke (width 0) (type default) (color 0 0 0 0))
-  )
   (wire (pts (xy 34.29 17.78) (xy 41.91 17.78))
     (stroke (width 0) (type default) (color 0 0 0 0))
@@
     (stroke (width 0) (type default) (color 0 0 0 0))
   )
-  (wire (pts (xy 73.66 55.88) (xy 73.66 74.93))
+  (wire (pts (xy 74.93 57.15) (xy 74.93 74.93))
     (stroke (width 0) (type default) (color 0 0 0 0))
   )
@@
     (stroke (width 0) (type default) (color 0 0 0 0))
   )
-  (wire (pts (xy 152.4 55.88) (xy 73.66 55.88))
+  (wire (pts (xy 152.4 57.15) (xy 74.93 57.15))
     (stroke (width 0) (type default) (color 0 0 0 0))
   )
@@
     (stroke (width 0) (type default) (color 0 0 0 0))
   )
-  (wire (pts (xy 109.22 78.74) (xy 113.03 78.74))
+  (wire (pts (xy 226.06 102.87) (xy 280.67 102.87))
     (stroke (width 0) (type default) (color 0 0 0 0))
   )
@@
     (stroke (width 0) (type default) (color 0 0 0 0))
   )
-  (wire (pts (xy 152.4 67.31) (xy 152.4 55.88))
+  (wire (pts (xy 152.4 67.31) (xy 152.4 57.15))
     (stroke (width 0) (type default) (color 0 0 0 0))
   )
@@
     (stroke (width 0) (type default) (color 0 0 0 0))
   )
-  (wire (pts (xy 109.22 46.99) (xy 109.22 78.74))
-    (stroke (width 0) (type default) (color 0 0 0 0))
-  )
   (wire (pts (xy 156.21 95.25) (xy 156.21 82.55))
     (stroke (width 0) (type default) (color 0 0 0 0))
   )
+  (wire (pts (xy 110.49 78.74) (xy 113.03 78.74))
+    (stroke (width 0) (type default) (color 0 0 0 0))
+  )
   (wire (pts (xy 113.03 107.95) (xy 107.95 107.95))
     (stroke (width 0) (type default) (color 0 0 0 0))
   )
+  (wire (pts (xy 153.67 107.95) (xy 280.67 107.95))
+    (stroke (width 0) (type default) (color 0 0 0 0))
+  )
   (wire (pts (xy 34.29 67.31) (xy 34.29 52.07))
     (stroke (width 0) (type default) (color 0 0 0 0))
@@
     (stroke (width 0) (type default) (color 0 0 0 0))
   )
-  (wire (pts (xy 106.68 76.2) (xy 111.76 76.2))
-    (stroke (width 0) (type default) (color 0 0 0 0))
-  )
   (wire (pts (xy 49.53 139.7) (xy 49.53 125.73))
     (stroke (width 0) (type default) (color 0 0 0 0))
@@
     (stroke (width 0) (type default) (color 0 0 0 0))
   )
-  (wire (pts (xy 236.22 102.87) (xy 236.22 40.64))
-    (stroke (width 0) (type default) (color 0 0 0 0))
-  )
   (wire (pts (xy 83.82 39.37) (xy 68.58 39.37))
     (stroke (width 0) (type default) (color 0 0 0 0))
@@
     (stroke (width 0) (type default) (color 0 0 0 0))
   )
-  (wire (pts (xy 236.22 40.64) (xy 111.76 40.64))
-    (stroke (width 0) (type default) (color 0 0 0 0))
-  )
   (wire (pts (xy 72.39 60.96) (xy 68.58 60.96))
     (stroke (width 0) (type default) (color 0 0 0 0))
   )
+  (wire (pts (xy 110.49 46.99) (xy 110.49 78.74))
+    (stroke (width 0) (type default) (color 0 0 0 0))
+  )
   (wire (pts (xy 24.13 81.28) (xy 20.32 81.28))
     (stroke (width 0) (type default) (color 0 0 0 0))
@@
     (stroke (width 0) (type default) (color 0 0 0 0))
   )
-  (wire (pts (xy 73.66 74.93) (xy 68.58 74.93))
+  (wire (pts (xy 74.93 74.93) (xy 68.58 74.93))
     (stroke (width 0) (type default) (color 0 0 0 0))
   )
@@
     (stroke (width 0) (type default) (color 0 0 0 0))
   )
-  (wire (pts (xy 41.91 17.78) (xy 106.68 17.78))
+  (wire (pts (xy 41.91 17.78) (xy 104.14 17.78))
     (stroke (width 0) (type default) (color 0 0 0 0))
   )
@@
     (stroke (width 0) (type default) (color 0 0 0 0))
   )
+  (wire (pts (xy 194.31 102.87) (xy 226.06 102.87))
+    (stroke (width 0) (type default) (color 0 0 0 0))
+  )
+  (wire (pts (xy 104.14 17.78) (xy 194.31 17.78))
+    (stroke (width 0) (type default) (color 0 0 0 0))
+  )
   (wire (pts (xy 38.1 125.73) (xy 34.29 125.73))
     (stroke (width 0) (type default) (color 0 0 0 0))
@@
     (stroke (width 0) (type default) (color 0 0 0 0))
   )
-  (wire (pts (xy 194.31 102.87) (xy 236.22 102.87))
-    (stroke (width 0) (type default) (color 0 0 0 0))
-  )
   (wire (pts (xy 78.74 118.11) (xy 68.58 118.11))
     (stroke (width 0) (type default) (color 0 0 0 0))
@@
     (stroke (width 0) (type default) (color 0 0 0 0))
   )
+  (text "To RPi GND" (at 269.24 101.6 0)
+    (effects (font (size 1.27 1.27)) (justify left bottom))
+  )
+  (text "To RPi GPIO1" (at 267.97 110.49 0)
+    (effects (font (size 1.27 1.27)) (justify left bottom))
+  )
+  (text "Pressure Mat" (at 40.64 151.13 0)
+    (effects (font (size 1.27 1.27)) (justify left bottom))
+  )
   (symbol (lib_id "Device:R_Variable_US") (at 68.58 129.54 0) (unit 1)
     (in_bom yes) (on_board yes) (fields_autoplaced)
@@
     (in_bom yes) (on_board yes) (fields_autoplaced)
     (property "Reference" "U2" (id 0) (at 204.47 86.3599 0)
-      (effects (font (size 1.27 1.27)) (justify left))
-    )
-    (property "Value" "NRF24L01_Breakout" (id 1) (at 204.47 88.8999 0)
+      (effects (font (size 1.27 1.27)) (justify left) hide)
+    )
+    (property "Value" "NRF24L01_Breakout" (id 1) (at 204.47 87.6299 0)
       (effects (font (size 1.27 1.27)) (justify left))
     )
@@
   (symbol (lib_id "Device:R_Pack06_SIP") (at 41.91 25.4 0) (unit 1)
     (in_bom yes) (on_board yes)
-    (property "Reference" "RN1" (id 0) (at 41.91 13.97 0))
+    (property "Reference" "RN1" (id 0) (at 41.91 13.97 0)
+      (effects (font (size 1.27 1.27)) hide)
+    )
     (property "Value" "R_Pack_SIP_1k" (id 1) (at 41.91 16.51 0))
     (property "Footprint" "Resistor_THT:R_Array_SIP12" (id 2) (at 66.675 25.4 90)
@@
     (in_bom yes) (on_board yes) (fields_autoplaced)
     (property "Reference" "U1" (id 0) (at 137.9094 151.13 0)
-      (effects (font (size 1.27 1.27)) (justify left))
-    )
-    (property "Value" "STM32F103RBTx" (id 1) (at 137.9094 153.67 0)
+      (effects (font (size 1.27 1.27)) (justify left) hide)
+    )
+    (property "Value" "STM32F103RB" (id 1) (at 137.9094 151.13 0)
       (effects (font (size 1.27 1.27)) (justify left))
     )
@@
     )
     (path "/b437c630-5fb9-453c-941b-b98bfdd865fc"
-      (reference "U1") (unit 1) (value "STM32F103RBTx") (footprint "Package_QFP:LQFP-64_10x10mm_P0.5mm")
+      (reference "U1") (unit 1) (value "STM32F103RB") (footprint "Package_QFP:LQFP-64_10x10mm_P0.5mm")
     )
     (path "/421d46db-68a7-4094-903c-2869122971ae"

Commit message: Updated schematic information on plot
Other:
- title: (none) -> STM32 System
Changed lines of the file:
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@@
 (kicad_sch (version 20211123) (generator eeschema)
   (paper "A4")
+  (title_block
+    (title "STM32 System")
+    (date "2023-03-24")
+  )
   (junction (at 68.58 147.32) (diameter 0) (color 0 0 0 0)
   )
