File: Ayden/Schematics/Wearable/Wearable.kicad_sch (KiCad schematic)
At the start: 6 parts

Commit message: Updated schematic information on plot
Other:
- title: (none) -> Wearable Device
Changed lines of the file:
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@@
 (kicad_sch (version 20230121) (generator eeschema)
   (paper "A4")
+  (title_block
+    (title "Wearable Device")
+    (date "2023-03-24")
+  )
   (junction (at 62.23 46.99) (diameter 0) (color 0 0 0 0)
   )
